File: KiCad_Projects/TX_50MHz_1W/TX_50MHz_1W.kicad_sch (KiCad schematic)
At the start: 51 parts, among them J1 AIL Stick, J10 I2C Exp / OLED, J11 ANT, J2 ELE Stick, J3 THR Stick, J4 RUD Stick, J5 AUX6, J6 AUX5, J7 AUX7, J8 V_BATT In (XT30), J9 5V Logic In, Q1 RD01MUS2 (1W PA), U1 ESP32-S3-WROOM-1-N16R8, U10 AP2112K-3.3TRG1, U2 Si5351A-B-GT, U3 BGS12SN6E6327XTSA1 (T/R SW), U4 SPF5043Z (LNA), U5 LT5560 (Mixer), U6 ADS1115IDGSR (0x48), U7 ADS1115IDGSR (0x49), U8 SH1106 1.3in OLED, U9 LMR33630BDDA, Y1 26.000MHz

Commit message: Re-tune TX antenna LPF cutoff away from 50MHz, verify with SPICE
Frequency-scaled the 7-pole ladder (L_new = L_old * fc_old/fc_new, same
for C, preserving shape and 50ohm impedance) to move the -3dB cutoff
from 49.1MHz to ~73MHz, then rounded to standard E12 parts:
  C2/C5: 120pF -> 82pF, C3/C4: 220pF -> 150pF, L3/L4/L5: 180nH -> 120nH

Added the three new values to Kraft6M.kicad_sym (library is shared
with the RX project; only new symbols were added, nothing existing
changed). Updated the 7 component instances in TX_50MHz_1W.kicad_sch
(lib_id, Value, and lib_symbols cache) accordingly.

Verified with ngspice: 50MHz now sits in a local S11 notch (VSWR 1.8,
S21 -0.37dB) instead of right on the filter's roll-off knee (was VSWR
10.4, S21 -5.0dB), while still keeping -37.6dB rejection at the 100MHz
2nd harmonic.

Co-Authored-By: Claude Sonnet 5 <noreply@anthropic.com>
Parts:
- C2, C5: value 120pF -> 82pF; symbol Kraft6M:C_120pF_0805 -> Kraft6M:C_82pF_0805
- C3, C4: value 220pF -> 150pF; symbol Kraft6M:C_220pF_0805 -> Kraft6M:C_150pF_0805
- L3, L4, L5: value 180nH -> 120nH; symbol Kraft6M:L_180nH_0805 -> Kraft6M:L_120nH_0805
Changed lines of the file:
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@@
 	)
 	(symbol
-		(lib_id "Kraft6M:C_220pF_0805")
+		(lib_id "Kraft6M:C_150pF_0805")
 		(at 224.79 76.2 90)
 		(unit 1)
@@
 			)
 		)
-		(property "Value" "220pF"
+		(property "Value" "150pF"
 			(at 231.14 76.2 90)
 			(show_name no)
@@
 	)
 	(symbol
-		(lib_id "Kraft6M:L_180nH_0805")
+		(lib_id "Kraft6M:L_120nH_0805")
 		(at 257.81 72.39 0)
 		(unit 1)
@@
 			)
 		)
-		(property "Value" "180nH"
+		(property "Value" "120nH"
 			(at 257.81 78.39 0)
 			(show_name no)
@@
 	)
 	(symbol
-		(lib_id "Kraft6M:L_180nH_0805")
+		(lib_id "Kraft6M:L_120nH_0805")
 		(at 214.63 72.39 0)
 		(unit 1)
@@
 			)
 		)
-		(property "Value" "180nH"
+		(property "Value" "120nH"
 			(at 214.63 78.39 0)
 			(show_name no)
@@
 	)
 	(symbol
-		(lib_id "Kraft6M:C_120pF_0805")
+		(lib_id "Kraft6M:C_82pF_0805")
 		(at 266.7 78.74 90)
 		(unit 1)
@@
 			)
 		)
-		(property "Value" "120pF"
+		(property "Value" "82pF"
 			(at 272.7 78.74 90)
 			(show_name no)
@@
 	)
 	(symbol
-		(lib_id "Kraft6M:C_120pF_0805")
+		(lib_id "Kraft6M:C_82pF_0805")
 		(at 201.93 74.93 90)
 		(unit 1)
@@
 			)
 		)
-		(property "Value" "120pF"
+		(property "Value" "82pF"
 			(at 207.93 74.93 90)
 			(show_name no)
@@
 	)
 	(symbol
-		(lib_id "Kraft6M:C_220pF_0805")
+		(lib_id "Kraft6M:C_150pF_0805")
 		(at 247.65 74.93 90)
 		(unit 1)
@@
 			)
 		)
-		(property "Value" "220pF"
+		(property "Value" "150pF"
 			(at 250.19 76.1999 90)
 			(show_name no)
@@
 	)
 	(symbol
-		(lib_id "Kraft6M:L_180nH_0805")
+		(lib_id "Kraft6M:L_120nH_0805")
 		(at 234.95 72.39 0)
 		(unit 1)
@@
 			)
 		)
-		(property "Value" "180nH"
+		(property "Value" "120nH"
 			(at 234.95 78.39 0)
 			(show_name no)

Commit message: Move receive chain to Si4463 upconversion; fix RX/TX schematic wiring
Replace the 10.7MHz IF + CD74HC4046A PLL discriminator with an LT5560
upconverter (Si5351 LO fixed at 118.2MHz) into a ~169MHz LC band-pass and
a Si4463-C2A-GM FSK packet receiver on SPI, on both the RX board and the
TX board's telemetry receiver. AX5043 rejected (out of production), CC1101
rejected (LO would exceed the Si5351's range).

Docs: design details, blueprints, BOMs, layout/power guides, firmware and
protocol specs, system docs and block diagrams updated to the new chain.

RX schematic: add Si4463 section; fix servo pins shorted onto one net,
I2C not reaching the ESP32, antenna bypassing the T/R switch, LNA not
reaching the mixer, and Si5351 CLK0 driving the mixer OUT- pin.

TX schematic: add Si4463 section; correct ESP32-S3-WROOM-1 pad numbers
(IO8-IO11 were on pads 11-14) in the schematic and Kraft6M library; AC-
ground LT5560 IN-/LO-/OUT- (were tied to GND); add SPF5043Z bias RFC and
DC block. Also includes the earlier USB_Interface sub-sheet split.

PCBs not yet updated from schematic; IF filter and AN643 match values TBD.

Co-Authored-By: Claude Opus 5.5 <noreply@anthropic.com>
Parts:
- removed FL1: 10.7MHz Murata SFE, Crystal:Resonator_SMD_Murata_SFECV-3Pin_6.9x2.9mm, symbol Kraft6M:10.7MHz_Filter
- added C25, C29: 10nF, Capacitor_SMD:C_0603_1608Metric, symbol Device:C
- added C26, C27, C28, C30: 100pF, Capacitor_SMD:C_0603_1608Metric, symbol Device:C
- added C31, C32, C33, C34, C35, C36, C37: TBD, Capacitor_SMD:C_0603_1608Metric, symbol Device:C
- added C38, C40: 100nF, Capacitor_SMD:C_0603_1608Metric, symbol Device:C
- added C39, C41: 1uF, Capacitor_SMD:C_0603_1608Metric, symbol Device:C
- added C42: 10pF, Capacitor_SMD:C_0603_1608Metric, symbol Device:C
- added L10, L11, L12, L13, L8, L9: TBD, Inductor_SMD:L_0603_1608Metric, symbol Device:L
- added L7: 1uH, Inductor_SMD:L_0805_2012Metric, symbol Device:L
- added R13: 10k, Resistor_SMD:R_0603_1608Metric, symbol Device:R
- added U13: Si4463-C2A-GM, Package_DFN_QFN:QFN-20-1EP_4x4mm_P0.5mm_EP2.6x2.6mm_ThermalVias, symbol RF:Si4463
- added Y2: 30MHz, Crystal:Crystal_SMD_3225-4Pin_3.2x2.5mm, symbol Device:Crystal_GND24
Connections:
- net +3V3: now also C25.1, C38.1, C39.1, C40.1, C41.1, C42.1, L7.1, L8.1, L9.1, R13.1, U13.6 (VDD), U13.8 (VDD); no longer U1.3 (EN)
- net 5V: no longer U10.3 (EN)
- net GND: now also C25.2, C27.2, C28.2, C29.2, C31.2, C33.2, C35.2, C37.2, C38.2, C39.2, C40.2, C41.2, C42.2, L10.2, L11.2, L12.2, U13.18 (GND), U13.21 (GND), Y2.2 (G), Y2.4 (G); no longer U5.2 (IN-), U5.6 (OUT-), U5.8 (LO-)
- net at J10.4 (P4), R4.2, U2.5 (SDA)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: now also U1.12 (IO8); no longer U1.11 (IO8)
- net at J10.3 (P3), R3.2, U2.4 (SCL)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: now also U1.17 (IO9); no longer U1.12 (IO9)
- net LNA_OUT: now reaches U4.3 (RFout)
- net LNA_OUT: now also C26.1, L7.2; no longer U5.1 (IN+)
- net at U3.6 (CTRL): now also U1.19 (IO11); no longer U1.14 (IO11)
- net IF_OUT_P: now reaches U5.5 (OUT+)
- net IF_OUT_P: now also C30.1, L8.2
- removed net ADC_IN: U1.13 (IO10)
- new net BOOT_IO0: U1.27 (IO0)
- new net EN: U1.3 (EN)
- new net IF_BPF_2: C32.2, C33.1, C34.1, L11.1
- new net IF_BPF_IN: C30.2, C31.1, C32.1, L10.1
- new net IF_BPF_OUT: C34.2, C35.1, C36.1, L12.1
- new net MIX_IN: C26.2, U5.1 (IN+)
- new net MIX_IN_N: C27.1, U5.2 (IN-)
- new net MIX_LO_N: C28.1, U5.8 (LO-)
- new net MIX_OUT_N: C29.1, L9.2, U5.6 (OUT-)
- new net SI_MISO: U1.22 (IO14), U13.13 (SDO)
- new net SI_MOSI: U1.21 (IO13), U13.14 (SDI)
- new net SI_RXN: C37.1, L13.2, U13.3 (RXn)
- new net SI_RXP: C36.2, L13.1, U13.2 (RXp)
- new net SI_SCLK: U1.20 (IO12), U13.12 (SCLK)
- new net SI_SDN: U1.10 (IO17), U13.1 (SDN)
- new net SI_XIN: U13.17 (XIN), Y2.1
- new net SI_XOUT: U13.16 (XOUT), Y2.3
- new net SI_nIRQ: R13.2, U1.9 (IO16), U13.11 (~{IRQ})
- new net SI_nSEL: U1.8 (IO15), U13.15 (~{SEL})
- new net U0RXD: U1.36 (RXD0)
- new net U0TXD: U1.37 (TXD0)
- no-connect marks 5 -> 13
Other:
- added sheet USB Interface (USB_Interface.kicad_sch)
- note added: "Telemetry receiver, Si4463 upconversion (2026-09-28). LT5560 up-converts 50MHz -> 168.3-169.2MHz (LO = Si5351 CLK1, 118.2MHz fixed, own PLL). L7/C25/C26: SPF5043Z bias RFC + DC block to mixer. C27-C29: LT5560 IN-/LO-/OUT- AC grounds (were tied straight to GND). L8/L9: LT5560 open-collector IF output feeds, value per LT5560 datasheet output network at 169MHz. L10-L12 / C31-C35: 3-pole top-C-couple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"
