File: KiCad_Projects/TX_50MHz_1W/TX_50MHz_1W.kicad_pcb (KiCad board)
At the start: 2 copper layers, 232.3 x 186.9 mm, 51 parts, among them J1 AIL Stick, J10 I2C Exp / OLED, J11 ANT, J2 ELE Stick, J3 THR Stick, J4 RUD Stick, J5 AUX6, J6 AUX5, J7 AUX7, J8 V_BATT In (XT30), J9 5V Logic In, Q1 RD01MUS2 (1W PA), U1 ESP32-S3-WROOM-1-N16R8, U10 AP2112K-3.3TRG1, U2 Si5351A-B-GT, U3 BGS12SN6E6327XTSA1 (T/R SW), U4 SPF5043Z (LNA), U5 LT5560 (Mixer), U6 ADS1115IDGSR (0x48), U7 ADS1115IDGSR (0x49), U8 SH1106 1.3in OLED, U9 LMR33630BDDA, Y1 26.000MHz

Commit message: Move receive chain to Si4463 upconversion; fix RX/TX schematic wiring
Replace the 10.7MHz IF + CD74HC4046A PLL discriminator with an LT5560
upconverter (Si5351 LO fixed at 118.2MHz) into a ~169MHz LC band-pass and
a Si4463-C2A-GM FSK packet receiver on SPI, on both the RX board and the
TX board's telemetry receiver. AX5043 rejected (out of production), CC1101
rejected (LO would exceed the Si5351's range).

Docs: design details, blueprints, BOMs, layout/power guides, firmware and
protocol specs, system docs and block diagrams updated to the new chain.

RX schematic: add Si4463 section; fix servo pins shorted onto one net,
I2C not reaching the ESP32, antenna bypassing the T/R switch, LNA not
reaching the mixer, and Si5351 CLK0 driving the mixer OUT- pin.

TX schematic: add Si4463 section; correct ESP32-S3-WROOM-1 pad numbers
(IO8-IO11 were on pads 11-14) in the schematic and Kraft6M library; AC-
ground LT5560 IN-/LO-/OUT- (were tied to GND); add SPF5043Z bias RFC and
DC block. Also includes the earlier USB_Interface sub-sheet split.

PCBs not yet updated from schematic; IF filter and AN643 match values TBD.

Co-Authored-By: Claude Opus 5.5 <noreply@anthropic.com>
Parts:
- moved J11 47.1 mm to (237.3, 35.0), turned to 180 degrees
- moved R3 37.4 mm to (108.5, 166.6)
- moved C6 20.1 mm to (38.4, 34.2)
- moved C13 14.1 mm to (189.0, 129.1)
- moved C11 10.7 mm to (134.3, 170.9)
- moved C17 9.93 mm to (189.0, 126.5)
- moved C12 9.88 mm to (176.9, 127.8)
- moved C8 8.92 mm to (107.3, 123.5)
- moved C9 8.32 mm to (63.9, 99.0)
- moved C15 8.20 mm to (196.8, 128.5)
- moved C16 7.87 mm to (201.1, 125.5)
- moved C7 7.87 mm to (91.2, 37.0)
- moved C10 2.13 mm to (51.2, 140.3)
Changed lines of the file:
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@@
 	(footprint "C_0603_1608Metric"
 		(layer "F.Cu")
-		(at 137.072621 181.275874)
+		(at 134.32 170.9)
 		(descr "Capacitor SMD 0603 (1608 Metric), square (rectangular) end terminal, IPC-7351 nominal, (Body size source: IPC-SM-782 page 76, https://www.pcb-3d.com/wordpress/wp-content/uploads/ipc-sm-782a_amendment_1_and_2.pdf)")
 		(tags "capacitor")
@@
 	(footprint "C_0603_1608Metric"
 		(layer "F.Cu")
-		(at 191.249 116.84)
+		(at 188.96 126.5)
 		(descr "Capacitor SMD 0603 (1608 Metric), square (rectangular) end terminal, IPC-7351 nominal, (Body size source: IPC-SM-782 page 76, https://www.pcb-3d.com/wordpress/wp-content/uploads/ipc-sm-782a_amendment_1_and_2.pdf)")
 		(tags "capacitor")
@@
 	(footprint "C_0603_1608Metric"
 		(layer "F.Cu")
-		(at 57.671 93.472)
+		(at 63.85 99.04)
 		(descr "Capacitor SMD 0603 (1608 Metric), square (rectangular) end terminal, IPC-7351 nominal, (Body size source: IPC-SM-782 page 76, https://www.pcb-3d.com/wordpress/wp-content/uploads/ipc-sm-782a_amendment_1_and_2.pdf)")
 		(tags "capacitor")
@@
 	(footprint "R_0603_1608Metric"
 		(layer "F.Cu")
-		(at 116.141 130.048)
+		(at 108.5 166.62)
 		(descr "Resistor SMD 0603 (1608 Metric), square (rectangular) end terminal, IPC-7351 nominal, (Body size source: IPC-SM-782 page 72, https://www.pcb-3d.com/wordpress/wp-content/uploads/ipc-sm-782a_amendment_1_and_2.pdf)")
 		(tags "resistor")
@@
 	(footprint "C_0603_1608Metric"
 		(layer "F.Cu")
-		(at 90.979164 29.185562)
+		(at 91.18 37.05)
 		(descr "Capacitor SMD 0603 (1608 Metric), square (rectangular) end terminal, IPC-7351 nominal, (Body size source: IPC-SM-782 page 76, https://www.pcb-3d.com/wordpress/wp-content/uploads/ipc-sm-782a_amendment_1_and_2.pdf)")
 		(tags "capacitor")
@@
 	(footprint "SMA_Amphenol_132289_EdgeMount"
 		(layer "F.Cu")
-		(at 190.193291 35)
+		(at 237.297622 35 180)
 		(descr "https://www.amphenolrf.com/library/download/link/link_id/595984/parent/132289/")
 		(tags "SMA")
@@
 	(footprint "C_0805_2012Metric"
 		(layer "F.Cu")
-		(at 183.029764 120.08625)
+		(at 176.9 127.83)
 		(descr "Capacitor SMD 0805 (2012 Metric), square (rectangular) end terminal, IPC-7351 nominal, (Body size source: IPC-SM-782 page 76, https://www.pcb-3d.com/wordpress/wp-content/uploads/ipc-sm-782a_amendment_1_and_2.pdf, https://docs.google.com/spreadsheets/d/1BsfQQcO9C6DZCsRaXUlFlo91Tg2WpOkGARC1WS5S8t0/edit?usp=sharing)")
 		(tags "capacitor")
@@
 	(footprint "C_0603_1608Metric"
 		(layer "F.Cu")
-		(at 19.244047 27.9235)
+		(at 38.36 34.25)
 		(descr "Capacitor SMD 0603 (1608 Metric), square (rectangular) end terminal, IPC-7351 nominal, (Body size source: IPC-SM-782 page 76, https://www.pcb-3d.com/wordpress/wp-content/uploads/ipc-sm-782a_amendment_1_and_2.pdf)")
 		(tags "capacitor")
@@
 	(footprint "C_0603_1608Metric"
 		(layer "F.Cu")
-		(at 201.065479 117.658)
+		(at 201.07 125.53)
 		(descr "Capacitor SMD 0603 (1608 Metric), square (rectangular) end terminal, IPC-7351 nominal, (Body size source: IPC-SM-782 page 76, https://www.pcb-3d.com/wordpress/wp-content/uploads/ipc-sm-782a_amendment_1_and_2.pdf)")
 		(tags "capacitor")
@@
 	(footprint "C_0603_1608Metric"
 		(layer "F.Cu")
-		(at 201.065479 121.43625)
+		(at 196.83 128.46)
 		(descr "Capacitor SMD 0603 (1608 Metric), square (rectangular) end terminal, IPC-7351 nominal, (Body size source: IPC-SM-782 page 76, https://www.pcb-3d.com/wordpress/wp-content/uploads/ipc-sm-782a_amendment_1_and_2.pdf)")
 		(tags "capacitor")
@@
 	(footprint "C_0603_1608Metric"
 		(layer "F.Cu")
-		(at 51.308 138.176)
+		(at 51.24 140.3)
 		(descr "Capacitor SMD 0603 (1608 Metric), square (rectangular) end terminal, IPC-7351 nominal, (Body size source: IPC-SM-782 page 76, https://www.pcb-3d.com/wordpress/wp-content/uploads/ipc-sm-782a_amendment_1_and_2.pdf)")
 		(tags "capacitor")
@@
 	(footprint "C_0603_1608Metric"
 		(layer "F.Cu")
-		(at 116.091 124.968)
+		(at 107.3 123.46)
 		(descr "Capacitor SMD 0603 (1608 Metric), square (rectangular) end terminal, IPC-7351 nominal, (Body size source: IPC-SM-782 page 76, https://www.pcb-3d.com/wordpress/wp-content/uploads/ipc-sm-782a_amendment_1_and_2.pdf)")
 		(tags "capacitor")
@@
 	(footprint "C_0603_1608Metric"
 		(layer "F.Cu")
-		(at 183.029764 116.308)
+		(at 188.96 129.1)
 		(descr "Capacitor SMD 0603 (1608 Metric), square (rectangular) end terminal, IPC-7351 nominal, (Body size source: IPC-SM-782 page 76, https://www.pcb-3d.com/wordpress/wp-content/uploads/ipc-sm-782a_amendment_1_and_2.pdf)")
 		(tags "capacitor")
