File: KiCad_Projects/TX_50MHz_1W/TX_Battery_Power.kicad_sch (KiCad schematic)
At the start: 0 parts

Commit message: broke up scheamatics into multiple files for easier navigation and organization. Added a new schematic page for organizing the schematics.  Added a new schematic page for the RX controller IO.  Added a new schematic page for the RX IF radio.  Added a new schematic page for the RX RF front end.  Added a new schematic page for the TX battery power.  Added a new schematic page for the TX controller RF.  Added a new schematic page for the TX telemetry IF.
Parts:
- added C12: 10uF, Capacitor_SMD:C_0805_2012Metric, symbol Kraft6M:C_10uF_0805
- added C13, C15, C16: 1uF, Capacitor_SMD:C_0603_1608Metric, symbol Kraft6M:C_1uF_0603
- added C14: 22uF, Capacitor_SMD:C_0805_2012Metric, symbol Kraft6M:C_22uF_0805
- added C17: 10nF, Capacitor_SMD:C_0603_1608Metric, symbol Kraft6M:C_10nF_0603
- added J8: V_BATT In (XT30), Connector_JST:JST_XH_B2B-XH-A_1x02_P2.50mm_Vertical, symbol Kraft6M:JST_XH_2Pin
- added J9: 5V Logic In, Connector_JST:JST_XH_B2B-XH-A_1x02_P2.50mm_Vertical, symbol Kraft6M:JST_XH_2Pin
- added L6: 10uH, Inductor_SMD:L_0805_2012Metric, symbol Kraft6M:L_10uH_0805
- added R1: 40.2k, Resistor_SMD:R_0603_1608Metric, symbol Kraft6M:R_40.2k_0603
- added R2: 10.2k, Resistor_SMD:R_0603_1608Metric, symbol Kraft6M:R_10.2k_0603
- added U10: AP2112K-3.3TRG1, Package_TO_SOT_SMD:SOT-23-5, symbol Kraft6M:AP2112K-3.3
- added U9: LMR33630BDDA, Package_SO:Texas_HSOP-8-1EP_3.9x4.9mm_P1.27mm_ThermalVias, symbol Kraft6M:LMR33630
Connections:
- net 5V: now also C14.2, C15.2, J9.1 (P1), L6.2, R1.1, U10.1 (VIN), U10.3 (EN)
- net V_BATT: now also C12.2, J8.1 (P1), U9.2 (VIN), U9.3 (EN)
- new net: R1.2, R2.1, U9.5 (FB)
- new net: C13.1, U9.6 (VCC)
- new net: C17.2, U9.7 (BOOT)
- new net: C17.1, L6.1, U9.8 (SW)
- new net +3V3: C16.2, U10.5 (VOUT)
- new net GND: C12.1, C13.2, C14.1, C15.1, C16.1, J8.2 (P2), J9.2 (P2), R2.2, U10.2 (GND), U9.1 (GND), U9.9 (GND)
- no-connect marks 0 -> 2
Other:
- removed sheet Battery + Power
- removed sheet Controller + TX RF
- removed sheet Telemetry IF
- removed sheet USB Interface
