File: KiCad_Projects/TX_50MHz_1W/TX_Controller_RF.kicad_sch (KiCad schematic)
At the start: 37 parts, among them J1 AIL Stick, J10 I2C Exp / OLED, J11 ANT, J2 ELE Stick, J3 THR Stick, J4 RUD Stick, J5 AUX6, J6 AUX5, J7 AUX7, Q1 RD01MUS2 (1W PA), U1 ESP32-S3-WROOM-1-N16R8, U2 Si5351A-B-GT, U3 BGS12SN6E6327XTSA1 (T/R SW), U4 SPF5043Z (LNA), U5 LT5560 (Mixer), U6 ADS1115IDGSR (0x48), U7 ADS1115IDGSR (0x49), U8 SH1106 1.3in OLED, Y1 26.000MHz

Commit message: udated scheamatic
Other:
- moved on the sheet: U4, U5

Commit message: lable correctly, local nets connected
Changed lines of the file:
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@@
 	(wire
 		(pts
-			(xy 83.82 67.31) (xy 87.63 67.31)
+			(xy 83.82 67.31) (xy 88.9 67.31)
 		)
 		(stroke
@@
 	(wire
 		(pts
-			(xy 224.79 43.18) (xy 242.57 43.18)
+			(xy 226.06 43.18) (xy 242.57 43.18)
 		)
 		(stroke
@@
 	(wire
 		(pts
-			(xy 262.89 38.1) (xy 261.62 38.1)
+			(xy 262.89 38.1) (xy 274.32 38.1)
 		)
 		(stroke
@@
 	(wire
 		(pts
-			(xy 262.89 35.56) (xy 261.62 35.56)
-		)
-		(stroke
-			(width 0)
-			(type default)
-		)
-	)
-	(wire
-		(pts
 			(xy 129.54 229.87) (xy 147.32 229.87)
 		)
@@
 	(wire
 		(pts
-			(xy 49.53 118.11) (xy 49.53 119.38)
-		)
-		(stroke
-			(width 0)
-			(type default)
-		)
-	)
-	(wire
-		(pts
 			(xy 185.42 100.33) (xy 185.42 127)
 		)
@@
 	(wire
 		(pts
+			(xy 76.2 40.64) (xy 76.2 46.99)
+		)
+		(stroke
+			(width 0)
+			(type default)
+		)
+	)
+	(wire
+		(pts
 			(xy 116.84 64.77) (xy 123.19 64.77)
 		)
@@
 	(wire
 		(pts
-			(xy 224.79 21.59) (xy 224.79 43.18)
+			(xy 226.06 34.29) (xy 226.06 43.18)
 		)
 		(stroke
@@
 	(wire
 		(pts
+			(xy 76.2 46.99) (xy 66.04 46.99)
+		)
+		(stroke
+			(width 0)
+			(type default)
+		)
+	)
+	(wire
+		(pts
 			(xy 105.41 80.01) (xy 83.82 80.01)
 		)
@@
 	(wire
 		(pts
-			(xy 49.53 119.38) (xy 57.15 119.38)
+			(xy 48.26 119.38) (xy 57.15 119.38)
 		)
 		(stroke
@@
 	(wire
 		(pts
-			(xy 87.63 21.59) (xy 224.79 21.59)
+			(xy 88.9 34.29) (xy 226.06 34.29)
 		)
 		(stroke
@@
 	(wire
 		(pts
+			(xy 274.32 35.56) (xy 262.89 35.56)
+		)
+		(stroke
+			(width 0)
+			(type default)
+		)
+	)
+	(wire
+		(pts
 			(xy 195.58 189.23) (xy 194.31 189.23)
 		)
@@
 	(wire
 		(pts
-			(xy 66.04 46.99) (xy 76.2 46.99)
+			(xy 76.2 40.64) (xy 52.07 40.64)
 		)
 		(stroke
@@
 	(wire
 		(pts
-			(xy 87.63 67.31) (xy 87.63 21.59)
+			(xy 88.9 67.31) (xy 88.9 34.29)
 		)
 		(stroke
@@
 	(hierarchical_label "MIX_OUT_N"
 		(shape bidirectional)
-		(at 261.62 38.1 0)
+		(at 274.32 38.1 0)
 		(effects
 			(font
@@
 	(hierarchical_label "IF_OUT_P"
 		(shape bidirectional)
-		(at 261.62 35.56 0)
+		(at 274.32 35.56 0)
 		(effects
 			(font
@@
 	(hierarchical_label "EN"
 		(shape bidirectional)
-		(at 49.53 118.11 180)
+		(at 48.26 119.38 180)
 		(effects
 			(font
@@
 	(symbol
 		(lib_id "power:GND")
-		(at 76.2 46.99 0)
+		(at 52.07 40.64 0)
 		(unit 1)
 		(body_style 1)
@@
 		(dnp no)
 		(property "Reference" "#PWR018"
-			(at 76.2 53.34 0)
+			(at 52.07 46.99 0)
 			(hide yes)
 			(show_name no)
@@
 		)
 		(property "Value" "GND"
-			(at 76.2 50.8 0)
+			(at 52.07 44.45 0)
 			(show_name no)
 			(do_not_autoplace no)
@@
 		)
 		(property "Footprint" ""
-			(at 76.2 46.99 0)
+			(at 52.07 40.64 0)
 			(hide yes)
 			(show_name no)
@@
 		)
 		(property "Datasheet" ""
-			(at 76.2 46.99 0)
+			(at 52.07 40.64 0)
 			(hide yes)
 			(show_name no)
@@
 		)
 		(property "Description" ""
-			(at 76.2 46.99 0)
+			(at 52.07 40.64 0)
 			(show_name no)
 			(do_not_autoplace no)
