File: KiCad_Projects/TX_50MHz_1W/TX_Telemetry_IF.kicad_sch (KiCad schematic)
At the start: 0 parts

Commit message: broke up scheamatics into multiple files for easier navigation and organization. Added a new schematic page for organizing the schematics.  Added a new schematic page for the RX controller IO.  Added a new schematic page for the RX IF radio.  Added a new schematic page for the RX RF front end.  Added a new schematic page for the TX battery power.  Added a new schematic page for the TX controller RF.  Added a new schematic page for the TX telemetry IF.
Parts:
- added C25, C29: 10nF, Capacitor_SMD:C_0603_1608Metric, symbol Device:C
- added C26, C27, C28, C30: 100pF, Capacitor_SMD:C_0603_1608Metric, symbol Device:C
- added C31, C32, C33, C34, C35, C36, C37: TBD, Capacitor_SMD:C_0603_1608Metric, symbol Device:C
- added C38, C40: 100nF, Capacitor_SMD:C_0603_1608Metric, symbol Device:C
- added C39, C41: 1uF, Capacitor_SMD:C_0603_1608Metric, symbol Device:C
- added C42: 10pF, Capacitor_SMD:C_0603_1608Metric, symbol Device:C
- added L10, L11, L12, L13, L8, L9: TBD, Inductor_SMD:L_0603_1608Metric, symbol Device:L
- added L7: 1uH, Inductor_SMD:L_0805_2012Metric, symbol Device:L
- added R13: 10k, Resistor_SMD:R_0603_1608Metric, symbol Device:R
- added U13: Si4463-C2A-GM, Package_DFN_QFN:QFN-20-1EP_4x4mm_P0.5mm_EP2.6x2.6mm_ThermalVias, symbol RF:Si4463
- added Y2: 30MHz, Crystal:Crystal_SMD_3225-4Pin_3.2x2.5mm, symbol Device:Crystal_GND24
Connections:
- net IF_OUT_P: now also C30.1, L8.2
- net LNA_OUT: now also C26.1, L7.2
- net MIX_IN: now also C26.2
- net MIX_IN_N: now also C27.1
- net MIX_LO_N: now also C28.1
- net MIX_OUT_N: now also C29.1, L9.2
- net SI_MISO: now also U13.13 (SDO)
- net SI_MOSI: now also U13.14 (SDI)
- net SI_SCLK: now also U13.12 (SCLK)
- net SI_SDN: now also U13.1 (SDN)
- net SI_nIRQ: now also R13.2, U13.11 (~{IRQ})
- net SI_nSEL: now also U13.15 (~{SEL})
- new net +3V3: C25.1, C38.1, C39.1, C40.1, C41.1, C42.1, L7.1, L8.1, L9.1, R13.1, U13.6 (VDD), U13.8 (VDD)
- new net GND: C25.2, C27.2, C28.2, C29.2, C31.2, C33.2, C35.2, C37.2, C38.2, C39.2, C40.2, C41.2, C42.2, L10.2, L11.2, L12.2, U13.18 (GND), U13.21 (GND), Y2.2 (G), Y2.4 (G)
- new net IF_BPF_2: C32.2, C33.1, C34.1, L11.1
- new net IF_BPF_IN: C30.2, C31.1, C32.1, L10.1
- new net IF_BPF_OUT: C34.2, C35.1, C36.1, L12.1
- new net SI_RXN: L13.2, U13.3 (RXn)
- new net SI_RXP: C36.2, L13.1, U13.2 (RXp)
- new net SI_XIN: C37.1, U13.17 (XIN)
- new net SI_XOUT: U13.16 (XOUT), Y2.3
- no-connect marks 0 -> 7
Other:
- removed sheet Battery + Power
- removed sheet Controller + TX RF
- removed sheet Telemetry IF
- removed sheet USB Interface
- note added: "Telemetry receiver, Si4463 upconversion (2026-09-28). LT5560 up-converts 50MHz -> 168.3-169.2MHz (LO = Si5351 CLK1, 118.2MHz fixed, own PLL). L7/C25/C26: SPF5043Z bias RFC + DC block to mixer. C27-C29: LT5560 IN-/LO-/OUT- AC grounds (were tied straight to GND). L8/L9: LT5560 open-collector IF output feeds, value per LT5560 datasheet output network at 169MHz. L10-L12 / C31-C35: 3-pole top-C-couple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"

Commit message: lable correctly, local nets connected
Other:
- moved on the sheet: C30, C31, C32, C33, C34, C35, C36, L10, L11, L12, L13, L8
