File: KiCad_Projects/TX_50MHz_1W/USB_Interface.kicad_sch (KiCad schematic)
At the start: 21 parts, among them J12 USB_C_Receptacle_USB2.0_14P, Q2 MMBT3904, Q3 MMBT3904, U11 CP2102N-A02-GQFN20, U12 MCP73831-2-OT

Commit message: broke up scheamatics into multiple files for easier navigation and organization. Added a new schematic page for organizing the schematics.  Added a new schematic page for the RX controller IO.  Added a new schematic page for the RX IF radio.  Added a new schematic page for the RX RF front end.  Added a new schematic page for the TX battery power.  Added a new schematic page for the TX controller RF.  Added a new schematic page for the TX telemetry IF.
Other:
- moved on the sheet: J12, R5, R6

Commit message: udated scheamatic
Connections:
- net +BATT: now also C24.2; no longer C24.1
- net GND: now also C24.1; no longer C24.2
Other:
- moved on the sheet: C24, R12

Commit message: lable correctly, local nets connected
Connections:
- net CC1_NET: now also J12.B5 (CC2); no longer J12.A5 (CC1)
- net CC2_NET: now also J12.A5 (CC1); no longer J12.B5 (CC2)
- net RTS_SIGNAL: now also R9.1
