File: KiCad_Projects/RX_50MHz_SDR/RX_50MHz_SDR.kicad_sch (KiCad schematic)
At the start: 44 parts, among them J1 ANTENNA, J10 SERVO6, J11 SERVO7, J12 SERVO8, J2 SERVO_5V_IN, J3 BATT+, J4 ESC+, J5 SERVO1, J6 SERVO2, J7 SERVO3, J8 SERVO4, J9 SERVO5, U1 ESP32-S3-WROOM-1, U2 LT5560EDD#PBF, U3 SPF5043Z, U4 Si5351A-B-GT, U5 AP2112K-3.3TRG1, U6 BGS12PL6, U7 INA219AIDCNR, Y1 26MHz

Commit message: Move receive chain to Si4463 upconversion; fix RX/TX schematic wiring
Replace the 10.7MHz IF + CD74HC4046A PLL discriminator with an LT5560
upconverter (Si5351 LO fixed at 118.2MHz) into a ~169MHz LC band-pass and
a Si4463-C2A-GM FSK packet receiver on SPI, on both the RX board and the
TX board's telemetry receiver. AX5043 rejected (out of production), CC1101
rejected (LO would exceed the Si5351's range).

Docs: design details, blueprints, BOMs, layout/power guides, firmware and
protocol specs, system docs and block diagrams updated to the new chain.

RX schematic: add Si4463 section; fix servo pins shorted onto one net,
I2C not reaching the ESP32, antenna bypassing the T/R switch, LNA not
reaching the mixer, and Si5351 CLK0 driving the mixer OUT- pin.

TX schematic: add Si4463 section; correct ESP32-S3-WROOM-1 pad numbers
(IO8-IO11 were on pads 11-14) in the schematic and Kraft6M library; AC-
ground LT5560 IN-/LO-/OUT- (were tied to GND); add SPF5043Z bias RFC and
DC block. Also includes the earlier USB_Interface sub-sheet split.

PCBs not yet updated from schematic; IF filter and AN643 match values TBD.

Co-Authored-By: Claude Opus 5.5 <noreply@anthropic.com>
Parts:
- removed FL1: 10.7MHz, Filter:Filter_Murata_SFECF-6, symbol Custom:FILTER3
- added C12: 4.7uF, Capacitor_SMD:C_0603_1608Metric, symbol Custom:CAP
- added C13, C15, C16: 0.1uF, Capacitor_SMD:C_0603_1608Metric, symbol Custom:CAP
- added C14, C26, C28: 1uF, Capacitor_SMD:C_0603_1608Metric, symbol Custom:CAP
- added C17: 100pF, Capacitor_SMD:C_0603_1608Metric, symbol Custom:CAP
- added C18, C19, C20, C21, C22, C23, C24: TBD, Capacitor_SMD:C_0603_1608Metric, symbol Custom:CAP
- added C25, C27: 100nF, Capacitor_SMD:C_0603_1608Metric, symbol Custom:CAP
- added C29: 10pF, Capacitor_SMD:C_0603_1608Metric, symbol Custom:CAP
- added J13: USB_C_Receptacle_USB2.0_14P, Connector_USB:USB_C_Receptacle_GCT_USB4085, symbol Connector:USB_C_Receptacle_USB2.0_14P
- added L10, L5, L6, L7, L8, L9: TBD, Inductor_SMD:L_0603_1608Metric, symbol Custom:IND
- added Q1, Q2: MMBT3904, Package_TO_SOT_SMD:SOT-23, symbol Transistor_BJT:MMBT3904
- added R3, R4: 5.1k, Resistor_SMD:R_0603_1608Metric, symbol Custom:RES
- added R5, R6, R7, R8, R9: 10k, Resistor_SMD:R_0603_1608Metric, symbol Custom:RES
- added U8: CP2102N-A02-GQFN20, Package_DFN_QFN:SiliconLabs_QFN-20-1EP_3x3mm_P0.5mm, symbol Interface_USB:CP2102N-Axx-xQFN20
- added U9: Si4463-C2A-GM, Package_DFN_QFN:QFN-20-1EP_4x4mm_P0.5mm_EP2.6x2.6mm_ThermalVias, symbol RF:Si4463
- added Y2: 30MHz, Crystal:Crystal_SMD_3225-4Pin_3.2x2.5mm, symbol Device:Crystal_GND24
Connections:
- net ADC_IF is gone; now on net SERVO1_SIG: U1.4 (IO4)
- net 3V3: now also C25.1, C26.1, C27.1, C28.1, C29.1, L5.1, L6.1, R9.1, U9.6 (VDD), U9.8 (VDD); no longer U1.3 (EN)
- net ANT: now also J1.1
- net GND: now also C12.2, C13.2, C14.2, C18.2, C20.2, C22.2, C24.2, C25.2, C26.2, C27.2, C28.2, C29.2, J13.A1 (GND), J13.A12 (GND), J13.B1 (GND), J13.B12 (GND), J13.SH (SHIELD), L7.2, L8.2, L9.2, Q1.2 (E), Q2.2 (E), R3.2, R4.2, U8.12 (GND), U8.15 (~{CTS}), U8.21 (GND), U8.3 (GND), U9.18 (GND), U9.21 (GND), Y2.2 (G), Y2.4 (G)
- net LNA_IN: now also D2.1, L1.1, U3.3 (RF_IN)
- net LO_CLK0: now also U4.6 (CLK0)
- net MIX_IN_N: now also C5.1
- net MIX_OUT_N: now also U2.6 (OUT-), L6.2
- net RF1_NET: now also C2.1
- net RX_EN: now also U1.23 (IO21)
- net SCL: now also U1.17 (IO9)
- net SDA: now also U1.12 (IO8)
- net SERVO1_SIG: now also J5.1 (SIG); no longer U1.9 (IO16)
- net SERVO2_SIG: now also U1.5 (IO5)
- net SERVO3_SIG: now also U1.6 (IO6)
- net SERVO4_SIG: now also U1.7 (IO7); no longer J12.1 (SIG)
- net SERVO5_SIG: now also U1.8 (IO15)
- net SERVO6_SIG: now also U1.9 (IO16)
- net SERVO7_SIG: now also U1.39 (IO1)
- net TELEM_TX_PRE: now also C1.2
- net TR_SW: now also U1.18 (IO10); no longer U2.1 (IN+)
- net VIN_LDO: no longer C10.1, L4.2, U5.1 (VIN), U5.3 (EN)
- net XTAL_B: no longer U4.3 (XB), Y1.2
- net IF_OUT_P: now reaches U2.5 (OUT+)
- net IF_OUT_P: now also C17.1, L5.2
- net MIX_IN: now reaches C3.2
- net MIX_IN: now also U2.1 (IN+)
- net SI_nIRQ: now reaches U1.10 (IO17)
- net SI_nIRQ: now also R9.2, U9.11 (~{IRQ})
- net SI_SDN: now reaches U1.11 (IO18)
- net SI_SDN: now also U9.1 (SDN)
- net SI_MOSI: now reaches U1.19 (IO11)
- net SI_MOSI: now also U9.14 (SDI)
- net SI_SCLK: now reaches U1.20 (IO12)
- net SI_SCLK: now also U9.12 (SCLK)
- new net: C16.2, Q2.1 (B), R8.2
- new net: C15.2, Q1.1 (B), R7.2
- new net: J13.A5 (CC1), R3.1
- new net: C10.1, L4.2, U5.1 (VIN), U5.3 (EN)
- new net: J13.B5 (CC2), R4.1
- new net: U4.3 (XB), Y1.2
- new net +3V3: C12.1, C13.1, R5.1, R6.1, U8.6 (VDD), U8.7 (VREGIN), U8.9 (~{RST})
- new net BOOT_IO0: Q2.3 (C), R6.2, U1.27 (IO0)
- new net DTR_SIGNAL: C15.1, R8.1, U8.1 (RS485/GPIO.1)
- new net EN: Q1.3 (C), R5.2, U1.3 (EN)
- new net IF_BPF_2: C19.2, C20.1, C21.1, L8.1
- new net IF_BPF_IN: C17.2, C18.1, C19.1, L7.1
- new net IF_BPF_OUT: C21.2, C22.1, C23.1, L9.1
- new net RTS_SIGNAL: C16.1, R7.1, U8.16 (~{RTS})
- new net SERVO8_SIG: J12.1 (SIG), U1.38 (IO2)
- new net SI_MISO: U1.21 (IO13), U9.13 (SDO)
- new net SI_RXN: C24.1, L10.2, U9.3 (RXn)
- new net SI_RXP: C23.2, L10.1, U9.2 (RXp)
- new net SI_XIN: U9.17 (XIN), Y2.1
- new net SI_XOUT: U9.16 (XOUT), Y2.3
- new net SI_nSEL: U1.22 (IO14), U9.15 (~{SEL})
- new net U0RXD: U1.36 (RXD0), U8.18 (TXD)
- new net U0TXD: U1.37 (TXD0), U8.17 (RXD)
- new net USB_DM: J13.A7 (D-), J13.B7 (D-), U8.5 (D-)
- new net USB_DP: J13.A6 (D+), J13.B6 (D+), U8.4 (D+)
- new net VBUS_5V: C14.1, J13.A4 (VBUS), J13.A9 (VBUS), J13.B4 (VBUS), J13.B9 (VBUS), U8.8 (VBUS)
- no-connect marks 0 -> 14
Other:
- note added: "169MHz IF + Si4463 receiver (2026-09-28). LT5560 up-converts 50MHz -> 168.3-169.2MHz (LO = Si5351 CLK0, 118.2MHz fixed). L5/L6: LT5560 open-collector IF output feeds, value per LT5560 datasheet output network at 169MHz. L7-L9 / C18-C22: 3-pole top-C-coupled LC band-pass, ~168.75MHz, ~3-5MHz BW, 50 ohm -- values TBD (design + SPICE). C23/L10/C24: Si4463 differential LNA match -- PLACEHOLDER topolo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"
- note added: "GPIO.1 must be OTP-configured as DTR via Silicon Labs Xpress Configurator before first use (factory default is RS485 direction control). Matches Espressif ESP32-S3-DevKitC-1 CP2102N config."
- moved on the sheet: C1, C10, C11, C9, C_bgsvdd1, D1, D2, D3, J3, J4, J8, L4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
