File: KiCad_Projects/RX_50MHz_SDR/RX_IF_Radio.kicad_sch (KiCad schematic)
At the start: 0 parts

Commit message: broke up scheamatics into multiple files for easier navigation and organization. Added a new schematic page for organizing the schematics.  Added a new schematic page for the RX controller IO.  Added a new schematic page for the RX IF radio.  Added a new schematic page for the RX RF front end.  Added a new schematic page for the TX battery power.  Added a new schematic page for the TX controller RF.  Added a new schematic page for the TX telemetry IF.
Parts:
- added C17: 100pF, Capacitor_SMD:C_0603_1608Metric, symbol Custom:CAP
- added C18, C19, C20, C21, C22, C23, C24: TBD, Capacitor_SMD:C_0603_1608Metric, symbol Custom:CAP
- added C25, C27: 100nF, Capacitor_SMD:C_0603_1608Metric, symbol Custom:CAP
- added C26, C28: 1uF, Capacitor_SMD:C_0603_1608Metric, symbol Custom:CAP
- added C29: 10pF, Capacitor_SMD:C_0603_1608Metric, symbol Custom:CAP
- added L10, L5, L6, L7, L8, L9: TBD, Inductor_SMD:L_0603_1608Metric, symbol Custom:IND
- added R9: 10k, Resistor_SMD:R_0603_1608Metric, symbol Custom:RES
- added U9: Si4463-C2A-GM, Package_DFN_QFN:QFN-20-1EP_4x4mm_P0.5mm_EP2.6x2.6mm_ThermalVias, symbol RF:Si4463
- added Y2: 30MHz, Crystal:Crystal_SMD_3225-4Pin_3.2x2.5mm, symbol Device:Crystal_GND24
Connections:
- net IF_OUT_P: now also C17.1, L5.2
- net MIX_OUT_N: now also L6.2
- net SI_MISO: now also U9.13 (SDO)
- net SI_MOSI: now also U9.14 (SDI)
- net SI_SCLK: now also U9.12 (SCLK)
- net SI_SDN: now also U9.1 (SDN)
- net SI_nIRQ: now also R9.2, U9.11 (~{IRQ})
- net SI_nSEL: now also U9.15 (~{SEL})
- new net 3V3: C25.1, C26.1, C27.1, C28.1, C29.1, L5.1, L6.1, R9.1, U9.6 (VDD), U9.8 (VDD)
- new net GND: C18.2, C20.2, C22.2, C24.2, C25.2, C26.2, C27.2, C28.2, C29.2, L7.2, L8.2, L9.2, U9.18 (GND), U9.21 (GND), Y2.2 (G), Y2.4 (G)
- new net IF_BPF_2: C19.2, C20.1, C21.1, L8.1
- new net IF_BPF_IN: C17.2, C18.1, C19.1, L7.1
- new net IF_BPF_OUT: C21.2, C22.1, C23.1, L9.1
- new net SI_RXN: C24.1, L10.2, U9.3 (RXn)
- new net SI_RXP: C23.2, L10.1, U9.2 (RXp)
- new net SI_XIN: U9.17 (XIN), Y2.1
- new net SI_XOUT: U9.16 (XOUT), Y2.3
- no-connect marks 0 -> 7
Other:
- removed sheet Controller - I/O
- removed sheet IF Radio
- removed sheet RF Front End
- note added: "169MHz IF + Si4463 receiver (2026-09-28). LT5560 up-converts 50MHz -> 168.3-169.2MHz (LO = Si5351 CLK0, 118.2MHz fixed). L5/L6: LT5560 open-collector IF output feeds, value per LT5560 datasheet output network at 169MHz. L7-L9 / C18-C22: 3-pole top-C-coupled LC band-pass, ~168.75MHz, ~3-5MHz BW, 50 ohm -- values TBD (design + SPICE). C23/L10/C24: Si4463 differential LNA match -- PLACEHOLDER topolo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"
- title: 50MHz RC Receiver - Auto-Generated Schematic -> (none)
