File: KiCad_Projects/RX_50MHz_SDR/RX_RF_Front_End.kicad_sch (KiCad schematic)
At the start: 0 parts

Commit message: broke up scheamatics into multiple files for easier navigation and organization. Added a new schematic page for organizing the schematics.  Added a new schematic page for the RX controller IO.  Added a new schematic page for the RX IF radio.  Added a new schematic page for the RX RF front end.  Added a new schematic page for the TX battery power.  Added a new schematic page for the TX controller RF.  Added a new schematic page for the TX telemetry IF.
Parts:
- added C1, C2, C3, C5, C8: 100pF, Capacitor_SMD:C_0603_1608Metric, symbol Custom:CAP
- added C4, C6, C7: 10nF, Capacitor_SMD:C_0603_1608Metric, symbol Custom:CAP
- added C_bgsvdd1: 0.1uF, Capacitor_SMD:C_0603_1608Metric, symbol Custom:CAP
- added D2, D3: BAV99, Package_TO_SOT_SMD:SOT-23, symbol Custom:DIODE
- added J1: ANTENNA, Connector_Coaxial:U.FL_Hirose_U.FL-R-SMT-1_Vertical, symbol Custom:HDR1
- added L1, L2: 220nH, Inductor_SMD:L_0603_1608Metric, symbol Custom:IND
- added L3: 1uH, Inductor_SMD:L_0805_2012Metric, symbol Custom:IND
- added R1, R2: 4.7k, Resistor_SMD:R_0603_1608Metric, symbol Custom:RES
- added U2: LT5560EDD#PBF, Package_DFN_QFN:DFN-8-1EP_3x3mm_P0.5mm_EP1.65x2.38mm, symbol Custom:LT5560
- added U3: SPF5043Z, ul_SPF5043Z:SPF5043Z_QOR, symbol Custom:SPF5043Z
- added U4: Si5351A-B-GT, Package_SO:MSOP-10_3x3mm_P0.5mm, symbol Custom:SI5351A
- added U6: BGS12PL6, Package_LGA:Infineon_PG-TSNP-6-10_0.7x1.1mm_0.7x1.1mm_P0.4mm, symbol Custom:BGS12PL6
- added Y1: 26MHz, Crystal:Crystal_SMD_3225-4Pin_3.2x2.5mm, symbol Custom:XTAL
Connections:
- net IF_OUT_P: now also U2.5 (OUT+)
- net MIX_OUT_N: now also C7.1, U2.6 (OUT-)
- net RX_EN: now also U2.3 (EN)
- net SCL: now also R2.2, U4.4 (SCL)
- net SDA: now also R1.2, U4.5 (SDA)
- net TR_SW: now also U6.4 (CTRL)
- new net: U4.3 (XB), Y1.2
- new net 3V3: C6.1, C_bgsvdd1.1, L3.2, R1.1, R2.1, U2.4 (VCC), U4.1 (VDD), U6.6 (VDD)
- new net ANT: J1.1, U6.5 (ANT)
- new net GND: C4.2, C5.2, C6.2, C7.2, C8.2, C_bgsvdd1.2, D2.2, D3.1, J1.2, L1.2, U2.9 (EP), U3.2 (GND), U3.4 (GND), U4.8 (GND), U6.2 (GND)
- new net LNA_IN: C2.2, D2.1, D3.2, L1.1, U3.3 (RF_IN)
- new net LNA_OUT_M: C3.1, L2.2
- new net LNA_OUT_VCC: C4.1, L2.1, L3.1, U3.1 (RF_OUT)
- new net LO_CLK0: U2.7 (LO+), U4.6 (CLK0)
- new net MIX_IN: C3.2, U2.1 (IN+)
- new net MIX_IN_N: C5.1, U2.2 (IN-)
- new net MIX_LO_N: C8.1, U2.8 (LO-)
- new net RF1_NET: C2.1, U6.3 (RF1)
- new net TELEM_TX_PRE: C1.2, U6.1 (RF2)
- new net TELEM_TX_PRE_B: C1.1, U4.7 (CLK1)
- new net XTAL_A: U4.2 (XA), Y1.1
Other:
- removed sheet Controller - I/O
- removed sheet IF Radio
- removed sheet RF Front End
- title: 50MHz RC Receiver - Auto-Generated Schematic -> (none)
